File: drum LMNC/TDrumer LMNC Clone/TDrumer LMNC Clone.kicad_pcb (KiCad board)
At the start: 2 copper layers, 141 parts, among them J1 Conn_02x05_Odd_Even, J10 HIBongoOut, J11 ClaveOut, J12 SnareOut, J13 MixOut, J2 KickTrig, J3 LOWBongoTrig, J4 HIBongoTrig, J5 ClaveTrig, J6 SnareTrig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

Commit message: add project
Parts:
- R16: footprint Resistor_THT:R_Axial_DIN0204_L3.6mm_D1.6mm_P7.62mm_Horizontal -> Resistor_THT:R_Axial_DIN0207_L6.3mm_D2.5mm_P10.16mm_Horizontal
- moved R12 133.5 mm to (165.1, 86.4), turned to 90 degrees
- moved L1 121.9 mm to (142.2, 50.8), turned to 90 degrees
- moved C5 100.3 mm to (157.5, 86.4), turned to 90 degrees
- moved U4 96.6 mm to (101.6, 45.7)
- moved R9 92.3 mm to (167.6, 83.8), turned to 90 degrees
- moved C7 90.3 mm to (155.0, 78.7)
- moved RV1 81.7 mm to (165.1, 71.1)
- moved R16 73.7 mm to (162.6, 78.7), turned to -90 degrees
- moved U3 59.3 mm to (170.2, 83.8)
- moved C9 51.5 mm to (144.8, 71.1), turned to 90 degrees
- moved RV2 47.6 mm to (157.5, 73.7), turned to 180 degrees
- moved C26 15.3 mm to (89.5, 76.2)
- moved U2 9.50 mm to (132.1, 94.0)
- moved Q2 1.58 mm to (135.2, 81.3)
- moved Q3 1.44 mm to (85.0, 129.5)
Routing:
- net (no net): track 2169.9 -> 2042.9 mm
- net GND: track 417.8 -> 450.8 mm
- net Net-(RV1-Pad1): track 0.00 -> 20.4 mm
- net Net-(C5-Pad1): track 0.00 -> 17.8 mm
- net Net-(C10-Pad1): track 0.00 -> 17.8 mm
- net Net-(C7-Pad2): track 0.00 -> 12.7 mm
- net Net-(R9-Pad2): track 0.00 -> 10.2 mm
- net Net-(C12-Pad1): track 0.00 -> 10.2 mm
- net Net-(C23-Pad1): track 0.00 -> 10.2 mm
- net Net-(C18-Pad1): track 0.00 -> 10.2 mm
- net Net-(C15-Pad2): track 0.00 -> 5.08 mm
- net Net-(C5-Pad2): track 0.00 -> 5.08 mm
- net Net-(C25-Pad2): track 0.00 -> 5.08 mm
- net Net-(C21-Pad2): track 0.00 -> 5.08 mm
- net +5V: track 0.00 -> 5.08 mm
